Commit message: change urdf

File: robots/hydrus/robots/quad/tilt_0deg_ce_15inch_202604/robot.urdf.xacro (robot description, xacro)
@@ -106,5 +106,5 @@
   <!--2.3-1 support ce spinal-->
   <xacro:extra_module name = "support_ce_spinal" parent = "support_livox" visible = "1"
-                      model_url = "package://hydrus/urdf/mesh/ver3/support_ce/support_ce_8R5.${mesh_ext}">
+                      model_url = "package://hydrus/urdf/mesh/ver3/support_ce/support_ce.${mesh_ext}">
     <origin xyz="0.0 0.0 0.0" rpy="0 0 0"/>
     <inertial>

File: robots/hydrus/urdf/common.xacro (robot description, xacro)
@@ -148,7 +148,7 @@
   </xacro:macro>
   <!-- support_ce -->
-  <xacro:macro name="support_ce_module" params="name parent *origin">
+  <xacro:macro name="support_ce_module" params="name parent model_url:=package://hydrus/urdf/mesh/ver3/support_ce/support_ce.${mesh_ext} *origin">
     <xacro:extra_module name="${name}" parent="${parent}" visible="1"
-                        model_url="package://hydrus/urdf/mesh/ver3/support_ce/support_ce_8R5.${mesh_ext}">
+                        model_url="${model_url}">
       <xacro:insert_block name="origin"/>
       <inertial>

File: robots/hydrus/urdf/link.urdf.xacro (robot description, xacro)
@@ -282,5 +282,6 @@
       <!-- support_ce4: link4 -->
       <xacro:if value="${self == 4}">
-        <xacro:support_ce_module name="support_ce4" parent="link4">
+        <xacro:support_ce_module name="support_ce4" parent="link4"
+                                 model_url="package://hydrus/urdf/mesh/ver3/support_painter/support_painter.${mesh_ext}">
           <origin xyz="${end_leg_offset} 0.000 0.01" rpy="0 0 0"/>
         </xacro:support_ce_module>

Commit message: change support

File: robots/hydrus/robots/quad/tilt_0deg_ce_15inch_202604/robot.urdf.xacro (robot description, xacro)
@@ -106,5 +106,5 @@
   <!--2.3-1 support ce spinal-->
   <xacro:extra_module name = "support_ce_spinal" parent = "support_livox" visible = "1"
-                      model_url = "package://hydrus/urdf/mesh/ver3/support_ce/support_ce.${mesh_ext}">
+                      model_url = "package://hydrus/urdf/mesh/ver3/support_ce/support_ce_8R5.${mesh_ext}">
     <origin xyz="0.0 0.0 0.0" rpy="0 0 0"/>
     <inertial>

File: robots/hydrus/urdf/common.xacro (robot description, xacro)
@@ -148,5 +148,5 @@
   </xacro:macro>
   <!-- support_ce -->
-  <xacro:macro name="support_ce_module" params="name parent model_url:=package://hydrus/urdf/mesh/ver3/support_ce/support_ce.${mesh_ext} *origin">
+  <xacro:macro name="support_ce_module" params="name parent model_url:=package://hydrus/urdf/mesh/ver3/support_ce/support_ce_8R5.${mesh_ext} *origin">
     <xacro:extra_module name="${name}" parent="${parent}" visible="1"
                         model_url="${model_url}">

File: robots/hydrus/urdf/link.urdf.xacro (robot description, xacro)
@@ -283,5 +283,5 @@
       <xacro:if value="${self == 4}">
         <xacro:support_ce_module name="support_ce4" parent="link4"
-                                 model_url="package://hydrus/urdf/mesh/ver3/support_painter/support_painter.${mesh_ext}">
+                                 model_url="package://hydrus/urdf/mesh/ver3/support_ce/support_ce_8R5.${mesh_ext}">
           <origin xyz="${end_leg_offset} 0.000 0.01" rpy="0 0 0"/>
         </xacro:support_ce_module>

Commit message: add side painter

File: robots/hydrus/robots/quad/tilt_0deg_ce_15inch_202604/robot.urdf.xacro (robot description, xacro)
@@ -10,5 +10,12 @@
   <xacro:hydrus_link links="4" self="2" rotor_direction="1"  with_battery = "0" tilt_mode="0" with_leg="1" mesh_ext="$(arg mesh_ext)" support_ce="1"/>
   <xacro:hydrus_link links="4" self="3" rotor_direction="-1" with_battery = "0" tilt_mode="0" with_leg="1" mesh_ext="$(arg mesh_ext)" support_ce="1"/>
-  <xacro:hydrus_link links="4" self="4" rotor_direction="1"  with_battery = "0" tilt_mode="0" with_leg="1" mesh_ext="$(arg mesh_ext)" support_ce="1"/>
+  <xacro:hydrus_link links="4" self="4" rotor_direction="1"  with_battery = "0" tilt_mode="0" with_leg="1" mesh_ext="$(arg mesh_ext)" support_ce="1"
+                     support_ce_model_url="package://hydrus/urdf/mesh/ver3/support_painter/support_painter_side.${mesh_ext}"
+                     support_ce4_inertial_origin_xyz="0.10434 0.00153 0.01788"
+                     support_ce4_inertial_origin_rpy="0 0 0"
+                     support_ce4_mass="0.1"
+                     support_ce4_ixx="0.00004181611" support_ce4_ixy="0.00001286954" support_ce4_ixz="0.00001494399"
+                     support_ce4_iyy="0.00057716187" support_ce4_iyz="0.00000031231"
+                     support_ce4_izz="0.00054349301"/>
   <!-- special battery arrangement -->
   <!-- <xacro:extra_module name = "bat1" parent = "link1" visible = "1"

File: robots/hydrus/urdf/common.xacro (robot description, xacro)
@@ -148,14 +148,14 @@
   </xacro:macro>
   <!-- support_ce -->
-  <xacro:macro name="support_ce_module" params="name parent model_url:=package://hydrus/urdf/mesh/ver3/support_ce/support_ce_8R5.${mesh_ext} *origin">
+  <xacro:macro name="support_ce_module" params="name parent model_url:=package://hydrus/urdf/mesh/ver3/support_ce/support_ce_8R5.${mesh_ext} inertial_origin_xyz:='0 0 0' inertial_origin_rpy:='0 0 0' mass:=0.001 ixx:=0.000001 ixy:=0.0 ixz:=0.0 iyy:=0.000001 iyz:=0.0 izz:=0.000001 *origin">
     <xacro:extra_module name="${name}" parent="${parent}" visible="1"
                         model_url="${model_url}">
       <xacro:insert_block name="origin"/>
       <inertial>
-        <origin xyz="0 0 0" rpy="0 0 0"/>
-        <mass value="0.001"/>
-        <inertia ixx="0.000001" ixy="0.0" ixz="0.0"
-                iyy="0.000001" iyz="0.0"
-                izz="0.000001"/>
+        <origin xyz="${inertial_origin_xyz}" rpy="${inertial_origin_rpy}"/>
+        <mass value="${mass}"/>
+        <inertia ixx="${ixx}" ixy="${ixy}" ixz="${ixz}"
+                iyy="${iyy}" iyz="${iyz}"
+                izz="${izz}"/>
       </inertial>
     </xacro:extra_module>

File: robots/hydrus/urdf/link.urdf.xacro (robot description, xacro)
@@ -3,5 +3,5 @@
     xmlns:xacro="http://www.ros.org/wiki/xacro" name="hydrus_link" >
   <!-- D-H kai description(different from prof.nakamura) -->
-  <xacro:macro name="hydrus_link" params="links self rotor_direction with_leg:=1 with_battery:=1 old_version:=0 tilt_mode:=0 tilt_angle:=0 prop_15inch:=0 mesh_ext:=dae support_ce:=0">
+  <xacro:macro name="hydrus_link" params="links self rotor_direction with_leg:=1 with_battery:=1 old_version:=0 tilt_mode:=0 tilt_angle:=0 prop_15inch:=0 mesh_ext:=dae support_ce:=0 support_ce_model_url:=package://hydrus/urdf/mesh/ver3/support_ce/support_ce_8R5.${mesh_ext} support_ce4_inertial_origin_xyz:='0 0 0' support_ce4_inertial_origin_rpy:='0 0 0' support_ce4_mass:=0.001 support_ce4_ixx:=0.000001 support_ce4_ixy:=0.0 support_ce4_ixz:=0.0 support_ce4_iyy:=0.000001 support_ce4_iyz:=0.0 support_ce4_izz:=0.000001">
     <xacro:if value="${old_version == 1}">
       <!-- link -->
@@ -283,5 +283,11 @@
       <xacro:if value="${self == 4}">
         <xacro:support_ce_module name="support_ce4" parent="link4"
-                                 model_url="package://hydrus/urdf/mesh/ver3/support_ce/support_ce_8R5.${mesh_ext}">
+                                 model_url="${support_ce_model_url}"
+                                 inertial_origin_xyz="${support_ce4_inertial_origin_xyz}"
+                                 inertial_origin_rpy="${support_ce4_inertial_origin_rpy}"
+                                 mass="${support_ce4_mass}"
+                                 ixx="${support_ce4_ixx}" ixy="${support_ce4_ixy}" ixz="${support_ce4_ixz}"
+                                 iyy="${support_ce4_iyy}" iyz="${support_ce4_iyz}"
+                                 izz="${support_ce4_izz}">
           <origin xyz="${end_leg_offset} 0.000 0.01" rpy="0 0 0"/>
         </xacro:support_ce_module>
