Commit message: add motorinfo_15inch and collision data

File: robots/delta/robots/quad/module_20260809/delta.gazebo.xacro (robot description, xacro)
@@ -5,4 +5,5 @@
   <xacro:arg name="module_visual_mesh_ext" default="stl" />
   <xacro:arg name="module_use_link_collision" default="true" />
+  <xacro:arg name="module_use_rotor_collision" default="false" />
   <xacro:include filename="$(find delta)/robots/quad/module_20260809/delta.urdf.xacro" />
   <!-- gazebo plugin for default controller and sensors -->

File: robots/delta/robots/quad/module_20260809/delta.urdf.xacro (robot description, xacro)
@@ -6,6 +6,8 @@
   <xacro:arg name="module_visual_mesh_ext" default="dae" />
   <xacro:arg name="module_use_link_collision" default="true" />
+  <xacro:arg name="module_use_rotor_collision" default="false" />
   <xacro:property name="module_visual_mesh_ext" value="$(arg module_visual_mesh_ext)" />
   <xacro:property name="module_use_link_collision" value="$(arg module_use_link_collision)" />
+  <xacro:property name="module_use_rotor_collision" value="$(arg module_use_rotor_collision)" />
   <xacro:property name="leg_length" value="0.207" />
   <xacro:property name="leg_radius" value="0.010" />

File: robots/delta/urdf/module_20260809/delta_link.urdf.xacro (robot description, xacro)
@@ -99,4 +99,11 @@
         </geometry>
       </visual>
+      <xacro:if value="${module_use_rotor_collision}">
+        <collision>
+          <geometry>
+            <cylinder radius="0.1905" length="0.01"/>
+          </geometry>
+        </collision>
+      </xacro:if>
     </link>
     <xacro:damping_factor link="thrust${self}" />
